File: kicad/projects/mixpower-path-nano-bq25620-board-r1/sheets/input-vbat.kicad_sch (KiCad schematic)
At the start: 22 parts, among them J6 BAT_HEADERS, J7 BATT, Q5 AO3401A, Q6 DMN3032LFDBQ, U6 TS5A3157, U7 DW01A, U8 MAX17055ETB

Commit message: feat: rework schematics and add proper calculations
Parts:
- removed Q5: AO3401A, Package_TO_SOT_SMD:SOT-23, symbol mixlib-discrete-mosfet:AO3401A
- added Q10: NTLJS17D0P03P8Z, mixlib-vendor-onsemi:vendor-onsemi-483av, symbol mixlib-discrete-mosfet:NTLJS17D0P03P8Z
- C32: now not fitted
- U7: value DW01A -> FS312F-G
Connections:
- net VBAT: now also Q10.4 (S), Q10.8 (S)
- net VBAT_IN: now also Q10.1 (D), Q10.2 (D), Q10.5 (D), Q10.6 (D), Q10.7 (D)
- net VBAT_IN_G: now also Q10.3 (G)
