File: kicad/projects/mixpower-path-nano-bq25620-board-r1/sheets/input-vbus.kicad_sch (KiCad schematic)
At the start: 28 parts, among them J5 USB_C_Receptacle_USB2.0_16P, Q4 Si1539CDL, U5 TPD8S300A

Commit message: feat: rework schematics and add proper calculations
Parts:
- TP1: value D+ -> D-
- TP2: value D- -> D+
Other:
- note added: "* ESD protection and filtering. * Maybe it needs proper calculation for this Pi-like filter... Or perhaps it matters not. * ESD is bidirectional because it's what I have in stock, but it can be replaced with a uni."
- note removed: "* ESD protection and filtering. * Maybe it needs proper calculation for this Pi-like filter... Or perhaps it matters not."
