File: kicad/projects/mixpower-path-nano-bq25620-board-r1/sheets/output-headers.kicad_sch (KiCad schematic)
At the start: 7 parts, among them J10 HAT, J11 DEBUG, J8 DATA_CONN, J9 DATA_HEADER

Commit message: feat: rework schematics and add proper calculations
Parts:
- added JP13: H1_SHIELD_TO_GND, Jumper:SolderJumper-2_P1.3mm_Open_Pad1.0x1.5mm, symbol Jumper:SolderJumper_2_Open
- added JP14: H2_SHIELD_TO_GND, Jumper:SolderJumper-2_P1.3mm_Open_Pad1.0x1.5mm, symbol Jumper:SolderJumper_2_Open
- added JP15: H3_SHIELD_TO_GND, Jumper:SolderJumper-2_P1.3mm_Open_Pad1.0x1.5mm, symbol Jumper:SolderJumper_2_Open
Connections:
- net GND: now also JP13.2 (B), JP14.2 (B), JP15.2 (B)
- net SHIELD: now also JP13.1 (A), JP14.1 (A), JP15.1 (A)
- net VBUS: now also J10.1 (Pin_1)
- net VOTG: no longer J10.1 (Pin_1)
Other:
- note added: "* For connection with a host (embedded MCU, PC, etc.). * Only USER Bus exposed (SCL_TX, SDA_RX), can be either I2C or UART. Internal Peripheral bus only accessible from the HAT Headers. * D+ and D- is bypassed to the host, but no MUX controls it. Host must communicate with the board to know when it's safe to establish USB communication. * ~{RST} and BOOT are useful for programming the host, espec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"
- note removed: "* For connection with a host (embedded SoC/MCU, PC, etc.). * Only USER Bus exposed (SCL_TX/SDA_RX), can be either I2C or UART. Internal Peripheral bus only accessible from the HAT Headers. * D+ and D- is bypassed to the host, but no MUX controls it. Host must communicate with the board to know when it's safe to use. * ~{RST} and BOOT are useful for programming the host, especially if they're ST M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"
- moved on the sheet: H1, H2, H3
