File: kicad/projects/mixpower-path-nano-bq25620-board-r1/sheets/ppc-bc.kicad_sch (KiCad schematic)
At the start: 21 parts, among them U14 BQ25620

Commit message: feat: rework schematics and add proper calculations
Parts:
- removed R65: 1M, Resistor_SMD:R_0402_1005Metric, symbol Device:R_Small
- added R82, R83, R84: 0, Resistor_SMD:R_0402_1005Metric, symbol Device:R_Small
Connections:
- net D+: now also R82.1; no longer U14.5 (D+)
- net D-: now also R83.1; no longer U14.4 (D-)
- net ~{QON}: now also R84.1; no longer U14.7 (~{QON})
- new net: R83.2, U14.4 (D-)
- new net: R84.2, U14.7 (~{QON})
- new net: R82.2, U14.5 (D+)
Other:
- note added: "* Considering L=(1uH * 0.7), D=0.5: - I_ripple = 3.571A - I_charge = 3A - I_saturation = 4.785 A"
- note added: "* Cutting USB is useful if switching to the STM32G0B1 MCUs, they have USB-BC detection."
- note added: "* Remove this resistor to disconnect the User Button from ~{QON}. This disables long-press reset and getting off ship mode on battery."
- note removed: "TODO: CALCULATE PROPER INDUCTOR VALUE (Considering ripple current, saturation current, etc.)"
- moved on the sheet: R67
