File: kicad/projects/mixpower-path-nano-bq25620-board-r1/sheets/soc-control.kicad_sch (KiCad schematic)
At the start: 18 parts, among them Q7 Si1026X, U10 TJ-S1615CY6TGLCCYRGY-A5, U9 STM32G071G8UxN

Commit message: feat: rework schematics and add proper calculations
Parts:
- R48, R49, R50: value 1.5k -> 1k
- U9: value STM32G071G8UxN -> STM32G071G8U6N
Other:
- note added: "* Two main LOGICAL buses are routed throughout the board: - USER: The USER bus is focused on controlling the board itself (SoC/MCU), e.g. setting up configuration, issuing commands, retrieving collected data, etc. It has a single physical bus with at most two wires, and can be multi-protocol (one chosen at a time). It can be a multi-master bus, when configured as I2C. As a rule, in this bus, the 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"
- note removed: "* Two main LOGICAL buses are routed throughout the board: - USER: The USER bus is focused on controlling the board itself (SoC/MCU), e.g. setting up configuration, issuing commands, retrieving collected data, etc. It has a single physical bus with at most two wires, and can be multi-protocol (one chosen at a time). It can be a multi-master bus, when configured as I2C. Also, as a rule, in this bus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"
- note removed: "TODO: REVISE THIS WHOLE DESCRIPTION!"
- moved on the sheet: R48, R49, R50, U10
