File: kicad/projects/mixpower-path-nano-bq25620-board-r1/subsheet__input-vbus.kicad_sch (KiCad schematic)
At the start: 28 parts, among them J5 USB_C_Receptacle_USB2.0_16P, Q4 Si1539CDL, U5 TPD8S300A

Commit message: fix: put all subsheets in root of the Kicad project, regenerate schematics plots
Parts:
- renumbered C25 to C10, C26 to C11, C27 to C12, C28 to C13, C29 to C14, C30 to C15, C24 to C9, D8 to D4, J5 to J2, Q4 to Q2, R24 to R11, R25 to R12, R26 to R13, R27 to R14, R28 to R15, R29 to R16, R30 to R17, R31 to R18, R32 to R19, R33 to R20, U5 to U2
Other:
- note added: "* ESD protection and filtering. * No proper calculation for this Pi-like filter... But perhaps it matters not. * ESD is bidirectional because it's what I have in stock, but it can be replaced with a unidirectional one with the same package."
- note removed: "* ESD protection and filtering. * Maybe it needs proper calculation for this Pi-like filter... Or perhaps it matters not. * ESD is bidirectional because it's what I have in stock, but it can be replaced with a uni."
- title: (none) -> mixpower-path-nano-bq25620-board
- moved on the sheet: JP6
