File: kicad/projects/mixpower-path-nano-bq25620-board-r1/subsheet__ppc-bc.kicad_sch (KiCad schematic)
At the start: 23 parts, among them U14 BQ25620

Commit message: fix: put all subsheets in root of the Kicad project, regenerate schematics plots
Parts:
- renumbered C45 to C21, C46 to C22, C47 to C23, C48 to C24, C49 to C25, C50 to C26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
Other:
- title: (none) -> mixpower-path-nano-bq25620-board
