File: kicad/projects/mixpower-path-nano-bq25620-board-r1/subsheet__vreg-3v3.kicad_sch (KiCad schematic)
At the start: 14 parts, among them U13 TPS63802

Commit message: fix: put all subsheets in root of the Kicad project, regenerate schematics plots
Parts:
- renumbered C43 to C31, C44 to C32, R58 to R39, R59 to R40, R60 to R41, R61 to R42, R62 to R43, R63 to R44, R64 to R45, TP8 to TP6, TP9 to TP7, TP10 to TP8, U13 to U7
Other:
- title: (none) -> mixpower-path-nano-bq25620-board
Changed lines of the file:
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@@
 	(generator_version "10.0")
 	(paper "A4")
+	(title_block
+		(title "mixpower-path-nano-bq25620-board")
+		(date "2026-04-05")
+		(rev "R1")
+	)
 	(rectangle
 		(start 134.62 93.98)
@@
 		(in_pos_files yes)
 		(dnp no)
-		(property "Reference" "C43"
+		(property "Reference" "C31"
 			(at 96.52 76.2062 0)
 			(show_name no)
@@
 			(project "mixpower-path-nano-bq25620-board-r1"
 				(path "/2e43857b-9bf9-460c-948c-ec2cf8a8d6b4/8d271180-8087-49c1-be7b-c6bf87d9e09d"
-					(reference "C43")
+					(reference "C31")
 					(unit 1)
 				)
@@
 		(in_pos_files yes)
 		(dnp no)
-		(property "Reference" "R63"
+		(property "Reference" "R44"
 			(at 163.83 95.2499 0)
 			(show_name no)
@@
 			(project "mixpower-path-nano-bq25620-board-r1"
 				(path "/2e43857b-9bf9-460c-948c-ec2cf8a8d6b4/8d271180-8087-49c1-be7b-c6bf87d9e09d"
-					(reference "R63")
+					(reference "R44")
 					(unit 1)
 				)
@@
 		(in_pos_files yes)
 		(dnp yes)
-		(property "Reference" "R58"
+		(property "Reference" "R39"
 			(at 107.95 96.5199 0)
 			(show_name no)
@@
 			(project "mixpower-path-nano-bq25620-board-r1"
 				(path "/2e43857b-9bf9-460c-948c-ec2cf8a8d6b4/8d271180-8087-49c1-be7b-c6bf87d9e09d"
-					(reference "R58")
+					(reference "R39")
 					(unit 1)
 				)
@@
 		(in_pos_files yes)
 		(dnp no)
-		(property "Reference" "C44"
+		(property "Reference" "C32"
 			(at 154.94 77.4762 0)
 			(show_name no)
@@
 			(project "mixpower-path-nano-bq25620-board-r1"
 				(path "/2e43857b-9bf9-460c-948c-ec2cf8a8d6b4/8d271180-8087-49c1-be7b-c6bf87d9e09d"
-					(reference "C44")
+					(reference "C32")
 					(unit 1)
 				)
@@
 		(in_pos_files yes)
 		(dnp no)
-		(property "Reference" "R59"
+		(property "Reference" "R40"
 			(at 107.95 106.6799 0)
 			(show_name no)
@@
 			(project "mixpower-path-nano-bq25620-board-r1"
 				(path "/2e43857b-9bf9-460c-948c-ec2cf8a8d6b4/8d271180-8087-49c1-be7b-c6bf87d9e09d"
-					(reference "R59")
+					(reference "R40")
 					(unit 1)
 				)
@@
 		(in_pos_files yes)
 		(dnp no)
-		(property "Reference" "R62"
+		(property "Reference" "R43"
 			(at 163.83 83.8199 0)
 			(show_name no)
@@
 			(project "mixpower-path-nano-bq25620-board-r1"
 				(path "/2e43857b-9bf9-460c-948c-ec2cf8a8d6b4/8d271180-8087-49c1-be7b-c6bf87d9e09d"
-					(reference "R62")
+					(reference "R43")
 					(unit 1)
 				)
@@
 		(in_pos_files yes)
 		(dnp no)
-		(property "Reference" "TP10"
+		(property "Reference" "TP8"
 			(at 160.02 111.7599 0)
 			(show_name no)
@@
 			(project "mixpower-path-nano-bq25620-board-r1"
 				(path "/2e43857b-9bf9-460c-948c-ec2cf8a8d6b4/8d271180-8087-49c1-be7b-c6bf87d9e09d"
-					(reference "TP10")
+					(reference "TP8")
 					(unit 1)
 				)
@@
 		(in_pos_files yes)
 		(dnp yes)
-		(property "Reference" "R64"
+		(property "Reference" "R45"
 			(at 171.45 90.1699 0)
 			(show_name no)
@@
 			(project "mixpower-path-nano-bq25620-board-r1"
 				(path "/2e43857b-9bf9-460c-948c-ec2cf8a8d6b4/8d271180-8087-49c1-be7b-c6bf87d9e09d"
-					(reference "R64")
+					(reference "R45")
 					(unit 1)
 				)
@@
 		(in_pos_files yes)
 		(dnp no)
-		(property "Reference" "R60"
+		(property "Reference" "R41"
 			(at 114.3 86.3599 0)
 			(show_name no)
@@
 			(project "mixpower-path-nano-bq25620-board-r1"
 				(path "/2e43857b-9bf9-460c-948c-ec2cf8a8d6b4/8d271180-8087-49c1-be7b-c6bf87d9e09d"
-					(reference "R60")
+					(reference "R41")
 					(unit 1)
 				)
@@
 		(in_pos_files yes)
 		(dnp no)
-		(property "Reference" "R61"
+		(property "Reference" "R42"
 			(at 163.83 77.4699 0)
 			(show_name no)
@@
 			(project "mixpower-path-nano-bq25620-board-r1"
 				(path "/2e43857b-9bf9-460c-948c-ec2cf8a8d6b4/8d271180-8087-49c1-be7b-c6bf87d9e09d"
-					(reference "R61")
+					(reference "R42")
 					(unit 1)
 				)
@@
 		(dnp no)
 		(fields_autoplaced yes)
-		(property "Reference" "#PWR077"
+		(property "Reference" "#PWR046"
 			(at 138.43 120.65 0)
 			(hide yes)
@@
 			(project "mixpower-path-nano-bq25620-board-r1"
 				(path "/2e43857b-9bf9-460c-948c-ec2cf8a8d6b4/8d271180-8087-49c1-be7b-c6bf87d9e09d"
-					(reference "#PWR077")
+					(reference "#PWR046")
 					(unit 1)
 				)
@@
 		(dnp no)
 		(fields_autoplaced yes)
-		(property "Reference" "#PWR079"
+		(property "Reference" "#PWR048"
 			(at 162.56 105.41 0)
 			(hide yes)
@@
 			(project "mixpower-path-nano-bq25620-board-r1"
 				(path "/2e43857b-9bf9-460c-948c-ec2cf8a8d6b4/8d271180-8087-49c1-be7b-c6bf87d9e09d"
-					(reference "#PWR079")
+					(reference "#PWR048")
 					(unit 1)
 				)
@@
 		(dnp no)
 		(fields_autoplaced yes)
-		(property "Reference" "#PWR076"
+		(property "Reference" "#PWR045"
 			(at 109.22 120.65 0)
 			(hide yes)
@@
 			(project "mixpower-path-nano-bq25620-board-r1"
 				(path "/2e43857b-9bf9-460c-948c-ec2cf8a8d6b4/8d271180-8087-49c1-be7b-c6bf87d9e09d"
-					(reference "#PWR076")
+					(reference "#PWR045")
 					(unit 1)
 				)
@@
 		(in_pos_files yes)
 		(dnp no)
-		(property "Reference" "TP9"
+		(property "Reference" "TP7"
 			(at 99.06 95.2499 0)
 			(show_name no)
@@
 			(project "mixpower-path-nano-bq25620-board-r1"
 				(path "/2e43857b-9bf9-460c-948c-ec2cf8a8d6b4/8d271180-8087-49c1-be7b-c6bf87d9e09d"
-					(reference "TP9")
+					(reference "TP7")
 					(unit 1)
 				)
@@
 		(dnp no)
 		(fields_autoplaced yes)
-		(property "Reference" "#PWR075"
+		(property "Reference" "#PWR044"
 			(at 99.06 86.36 0)
 			(hide yes)
@@
 			(project "mixpower-path-nano-bq25620-board-r1"
 				(path "/2e43857b-9bf9-460c-948c-ec2cf8a8d6b4/8d271180-8087-49c1-be7b-c6bf87d9e09d"
-					(reference "#PWR075")
+					(reference "#PWR044")
 					(unit 1)
 				)
@@
 		(in_pos_files yes)
 		(dnp no)
-		(property "Reference" "TP8"
+		(property "Reference" "TP6"
 			(at 99.06 85.0899 0)
 			(show_name no)
@@
 			(project "mixpower-path-nano-bq25620-board-r1"
 				(path "/2e43857b-9bf9-460c-948c-ec2cf8a8d6b4/8d271180-8087-49c1-be7b-c6bf87d9e09d"
-					(reference "TP8")
+					(reference "TP6")
 					(unit 1)
 				)
@@
 		(dnp no)
 		(fields_autoplaced yes)
-		(property "Reference" "U13"
+		(property "Reference" "U7"
 			(at 127 73.66 0)
 			(show_name no)
@@
 			(project "mixpower-path-nano-bq25620-board-r1"
 				(path "/2e43857b-9bf9-460c-948c-ec2cf8a8d6b4/8d271180-8087-49c1-be7b-c6bf87d9e09d"
-					(reference "U13")
+					(reference "U7")
 					(unit 1)
 				)
@@
 		(dnp no)
 		(fields_autoplaced yes)
-		(property "Reference" "#PWR078"
+		(property "Reference" "#PWR047"
 			(at 157.48 87.63 0)
 			(hide yes)
@@
 			(project "mixpower-path-nano-bq25620-board-r1"
 				(path "/2e43857b-9bf9-460c-948c-ec2cf8a8d6b4/8d271180-8087-49c1-be7b-c6bf87d9e09d"
-					(reference "#PWR078")
+					(reference "#PWR047")
 					(unit 1)
 				)
